Commit message: jackal sensor

File: entities/robots/jackal/urdf/jackal.urdf.xacro (robot description, xacro)
@@ -191,4 +191,32 @@
     <child link="imu_link" />
   </joint>
+    <!-- LiDAR Link -->
+  <link name="lidar_link">
+    <inertial>
+      <origin xyz="0 0 0" rpy="0 0 0"/>
+      <mass value="0.1"/>
+      <inertia ixx="1e-5" ixy="0" ixz="0" iyy="1e-5" iyz="0" izz="1e-5"/>
+    </inertial>
+    <visual>
+      <origin xyz="0 0 0" rpy="0 0 0"/>
+      <geometry>
+        <cylinder radius="0.05" length="0.1"/>
+      </geometry>
+      <material name="black"/>
+    </visual>
+    <collision>
+      <origin xyz="0 0 0" rpy="0 0 0"/>
+      <geometry>
+        <cylinder radius="0.05" length="0.1"/>
+      </geometry>
+    </collision>
+  </link>
+  <!-- LiDAR Joint -->
+  <joint name="lidar_joint" type="fixed">
+    <parent link="chassis_link"/>
+    <child link="lidar_link"/>
+    <!-- Adjust the position below to place the LiDAR appropriately -->
+    <origin xyz="0.0 0.0 ${chassis_height/2 + 0.05}" rpy="0 0 0"/>
+  </joint>
   <!-- TODO: Same note as applies to imu_link -->
   <link name="navsat_link">

Commit message: jackal is working and im malding

File: entities/robots/jackal/urdf/jackal.urdf.xacro (robot description, xacro)
@@ -191,30 +191,32 @@
     <child link="imu_link" />
   </joint>
+  <frame name="lidar_frame" attached_to="chassis_link">
+    <pose>0.0 0.0 ${chassis_height/2 + 0.05} 0 0 0</pose>
+  </frame>
   <link name="lidar_link">
-    <inertial>
-      <origin xyz="0 0 0" rpy="0 0 0"/>
-      <mass value="0.1"/>
-      <inertia ixx="1e-5" ixy="0" ixz="0" iyy="1e-5" iyz="0" izz="1e-5"/>
-    </inertial>
-    <visual>
-      <origin xyz="0 0 0" rpy="0 0 0"/>
-      <geometry>
-        <cylinder radius="0.05" length="0.1"/>
-      </geometry>
-      <material name="black"/>
-    </visual>
-    <collision>
-      <origin xyz="0 0 0" rpy="0 0 0"/>
-      <geometry>
-        <cylinder radius="0.05" length="0.1"/>
-      </geometry>
-    </collision>
+      <inertial>
+          <origin xyz="0 0 0" rpy="0 0 0"/>
+          <mass value="0.1"/>
+          <inertia ixx="1e-5" ixy="0" ixz="0" iyy="1e-5" iyz="0" izz="1e-5"/>
+      </inertial>
+      <visual>
+          <origin xyz="0 0 0" rpy="0 0 0"/>
+          <geometry>
+              <cylinder radius="0.05" length="0.1"/>
+          </geometry>
+          <material name="black"/>
+      </visual>
+      <collision>
+          <origin xyz="0 0 0" rpy="0 0 0"/>
+          <geometry>
+              <cylinder radius="0.05" length="0.1"/>
+          </geometry>
+      </collision>
   </link>
   <!-- Fixed joint to attach the LiDAR to the chassis -->
   <joint name="lidar_joint" type="fixed">
-    <parent link="chassis_link"/>
-    <child link="lidar_link"/>
-    <!-- Adjust xyz to place LiDAR where you want it -->
-    <origin xyz="0.0 0.0 ${chassis_height/2 + 0.05}" rpy="0 0 0"/>
+      <parent link="chassis_link"/>
+      <child link="lidar_link"/>
+      <origin xyz="0.0 0.0 ${chassis_height/2 + 0.05}" rpy="0 0 0"/>
   </joint>
   <!-- TODO: Same note as applies to imu_link -->

File: entities/robots/turtlebot4/urdf/sensors/rplidar.urdf.xacro (robot description, xacro)
@@ -30,9 +30,4 @@
   </link>
   <gazebo reference="${name}_link">
-    <!--
-      GPU Ray sensor plugin only supports 180 degrees, so limit to the "front" arc only
-      The lidar is actually mounted sideways on the robot, with +x to the left, so the
-      front arc is actually 0 to -pi
-    -->
     <xacro:ray_sensor sensor_name="${name}" gazebo="${gazebo}"
                   update_rate="62.0" visualize="1"
