Commit message: house1

File: entities/robots/jackal/urdf/jackal.urdf (robot description, URDF)
Before this commit: robot jackal, 13 links, 12 joints
Links:
- added link lidar_link, mass 0.1; collision cylinder length=0.1 radius=0.05; visual cylinder length=0.1 radius=0.05
Joints:
- added joint lidar_joint: type fixed, parent chassis_link, child lidar_link, origin xyz=0.0 0.0 0.14200000000000002 rpy=0 0 0
